Commit message: feat(model): Added a simple box geometry to the robot model.

File: src/my_robot_description/urdf/my_robot.urdf (robot description, URDF)
Before this commit: robot my_robot, 0 links, 0 joints
Links:
- added link base_link; visual box size=0.6 0.4 0.2

Commit message: feat(robot): Created my_robot.urdf file and completed the robot model.

File: src/my_robot_description/urdf/my_robot.urdf (robot description, URDF)
Before this commit: robot my_robot, 1 links, 0 joints
Links:
- added link back_left_caster_wheel_link; visual sphere radius=${caster_wheel_radius}
- added link back_right_caster_wheel_link; visual sphere radius=${caster_wheel_radius}
- added link left_wheel_link; visual cylinder length=${wheel_length} radius=${wheel_radius}
- added link pre_left_caster_wheel_link; visual sphere radius=${caster_wheel_radius}
- added link pre_right_caster_wheel_link; visual sphere radius=${caster_wheel_radius}
- added link right_wheel_link; visual cylinder length=${wheel_length} radius=${wheel_radius}
- link base_link: geometry visual box size=${base_with} ${base_length} ${base_height}
Joints:
- added joint base_back_left_caster_wheel_joint: type continuous, parent base_link, child back_left_caster_wheel_link, origin xyz=${(caster_wheel_radius * 6) - (caster_wheel_radius)}                         ${-(base_length / 2) + (caster_wheel_radius)}                         ${-3 * (caster_wheel_radius)} rpy=0 0 0, axis 0 1 0
- added joint base_back_right_caster_wheel_joint: type continuous, parent base_link, child back_right_caster_wheel_link, origin xyz=${(caster_wheel_radius * 6) - (caster_wheel_radius)}                         ${(base_length / 2) - (caster_wheel_radius)}                         ${-3 * (caster_wheel_radius)} rpy=0 0 0, axis 0 1 0
- added joint base_left_wheel_joint: type continuous, parent base_link, child left_wheel_link, origin xyz=${- (base_height / 2) + (wheel_radius) }                        ${((base_length / 2) + (wheel_length / 2))}                        ${- wheel_radius} rpy=0 0 0, axis 0 1 0
- added joint base_pre_left_caster_wheel_joint: type continuous, parent base_link, child pre_left_caster_wheel_link, origin xyz=${-(caster_wheel_radius * 6) + (caster_wheel_radius)}                         ${-(base_length / 2) + (caster_wheel_radius)}                         ${-3 * (caster_wheel_radius)} rpy=0 0 0, axis 0 1 0
- added joint base_pre_right_caster_wheel_joint: type continuous, parent base_link, child pre_right_caster_wheel_link, origin xyz=${-(caster_wheel_radius * 6) + (caster_wheel_radius)}                         ${(base_length / 2) - (caster_wheel_radius)}                         ${-3 * (caster_wheel_radius)} rpy=0 0 0, axis 0 1 0
- added joint base_right_wheel_joint: type continuous, parent base_link, child right_wheel_link, origin xyz=${- (base_height / 2) + (wheel_radius) }                        ${-((base_length / 2) + (wheel_length / 2))}                        ${- wheel_radius} rpy=0 0 0, axis 0 1 0

Commit message: refactor(code): The code has been refactored thanks to the macro inside xacro and the use of prefixes to reduce code repetition.

File: src/my_robot_description/urdf/my_robot.urdf (robot description, URDF)
Before this commit: robot my_robot, 7 links, 6 joints
Links:
- removed link back_left_caster_wheel_link
- removed link back_right_caster_wheel_link
- removed link left_wheel_link
- removed link pre_left_caster_wheel_link
- removed link pre_right_caster_wheel_link
- removed link right_wheel_link

Commit message: fix: Fixed bug caused by missing $ sign

File: src/my_robot_description/urdf/my_robot.urdf (robot description, URDF)
Before this commit: robot my_robot, 1 links, 6 joints
Links:
- added link base_footprint
Joints:
- added joint base_joint: type fixed, parent base_footprint, child base_link, origin xyz=0 0 ${(base_height / 2) + wheel_radius} rpy=0 0 0
