Commit message: feat(robot_model): Camera fixed to base_link.

File: src/my_alfa_robot_description/urdf/camera.xacro (robot description, xacro)
@@ -27,3 +27,9 @@
                                      elde etmiş olurum. 2* genişleterek bu durumu düzeltemiş olurum.-->
     </link>
+       <!-- Kamera ve base_link arasında sabit bağlantı (joint) -->
+    <joint name="base_camera_joint" type="fixed">
+        <parent link="base_link"/>
+        <child link="camera_link"/>
+        <origin xyz="0.3 0 0" rpy="0 0 0"/>
+    </joint>
 </robot>
